Commit message: hubo.urdf: add header-like comments

File: hubo_description/urdf/hubo.urdf (robot description, URDF)
Before this commit: robot huboplus, 59 links, 58 joints
Joints:
- joint HNP: type revolute -> fixed

Commit message: make most of the joints fixed
make all joints other than those on legs and arms fixed

File: hubo_description/urdf/hubo.urdf (robot description, URDF)
Before this commit: robot huboplus, 59 links, 58 joints
Joints:
- joint WST: type revolute -> fixed
- joint leftIndexKnuckle1: type revolute -> fixed
- joint leftIndexKnuckle2: type revolute -> fixed
- joint leftIndexKnuckle3: type revolute -> fixed
- joint leftMiddleKnuckle1: type revolute -> fixed
- joint leftMiddleKnuckle2: type revolute -> fixed
- joint leftMiddleKnuckle3: type revolute -> fixed
- joint leftPinkyKnuckle1: type revolute -> fixed
- joint leftPinkyKnuckle2: type revolute -> fixed
- joint leftPinkyKnuckle3: type revolute -> fixed
- joint leftRingKnuckle1: type revolute -> fixed
- joint leftRingKnuckle2: type revolute -> fixed
- joint leftRingKnuckle3: type revolute -> fixed
- joint leftThumbKnuckle1: type revolute -> fixed
- joint leftThumbKnuckle2: type revolute -> fixed
- joint leftThumbKnuckle3: type revolute -> fixed
- joint rightIndexKnuckle1: type revolute -> fixed
- joint rightIndexKnuckle2: type revolute -> fixed
- joint rightIndexKnuckle3: type revolute -> fixed
- joint rightMiddleKnuckle1: type revolute -> fixed
- joint rightMiddleKnuckle2: type revolute -> fixed
- joint rightMiddleKnuckle3: type revolute -> fixed
- joint rightPinkyKnuckle1: type revolute -> fixed
- joint rightPinkyKnuckle2: type revolute -> fixed
- joint rightPinkyKnuckle3: type revolute -> fixed
- joint rightRingKnuckle1: type revolute -> fixed
- joint rightRingKnuckle2: type revolute -> fixed
- joint rightRingKnuckle3: type revolute -> fixed
- joint rightThumbKnuckle1: type revolute -> fixed
- joint rightThumbKnuckle2: type revolute -> fixed
- joint rightThumbKnuckle3: type revolute -> fixed
