Commit message: replace hubo.urdf with .xacro based definition, add kinect
kinect has been taken from the pr2_description package and modified

File: hubo_description/urdf/hubo.urdf.xacro (robot description, xacro)
@@ -1,9 +1,8 @@
-<?xml version="1.0" ?>
-<!-- =================================================================================== -->
-<!-- |    This document was autogenerated by xacro from huboplus.xacro                 | -->
-<!-- |    EDITING THIS FILE BY HAND IS NOT RECOMMENDED                                 | -->
-<!-- =================================================================================== -->
-<robot name="huboplus" xmlns:xacro="http://www.ros.org/wiki/xacro">
-  <!-- Links - - - - - - - - - - - - - - - - - - - - - - - - -->
+<?xml version="1.0"?>
+<robot xmlns:sensor="http://playerstage.sourceforge.net/gazebo/xmlschema/#sensor"
+       xmlns:controller="http://playerstage.sourceforge.net/gazebo/xmlschema/#controller"
+       xmlns:interface="http://playerstage.sourceforge.net/gazebo/xmlschema/#interface"
+       xmlns:xacro="http://ros.org/wiki/xacro">
+<xacro:macro name="hubo">
   <link name="Body_Torso">
     <inertial>
@@ -1803,3 +1802,4 @@
     <pose>0 0 1 0 0 0</pose>
   </gazebo>
+</xacro:macro>
 </robot>

Commit message: increase right hand joints' effort limit

File: hubo_description/urdf/hubo.urdf.xacro (robot description, xacro)
@@ -1363,5 +1363,5 @@
     <child link="Body_RSP"/>
     <axis xyz="0 1 0"/>
-    <limit effort="10.0" lower="-3.14158" upper="3.14158" velocity="1.0"/>
+    <limit effort="50.0" lower="-3.14158" upper="3.14158" velocity="1.0"/>
   </joint>
   <joint name="RSR" type="revolute">
@@ -1370,5 +1370,5 @@
     <child link="Body_RSR"/>
     <axis xyz="1 0 0"/>
-    <limit effort="10.0" lower="-3.14158" upper="0" velocity="1.0"/>
+    <limit effort="50.0" lower="-3.14158" upper="0" velocity="1.0"/>
   </joint>
   <joint name="RSY" type="revolute">
@@ -1377,5 +1377,5 @@
     <child link="Body_RSY"/>
     <axis xyz="0 0 1"/>
-    <limit effort="10.0" lower="-3.14158" upper="3.14158" velocity="1.0"/>
+    <limit effort="50.0" lower="-3.14158" upper="3.14158" velocity="1.0"/>
   </joint>
   <joint name="REP" type="revolute">
@@ -1384,5 +1384,5 @@
     <child link="Body_REP"/>
     <axis xyz="0 1 0"/>
-    <limit effort="10.0" lower="-2.49582" upper="0.0698132" velocity="1.0"/>
+    <limit effort="50.0" lower="-2.49582" upper="0.0698132" velocity="1.0"/>
   </joint>
   <joint name="RWY" type="revolute">
@@ -1391,5 +1391,5 @@
     <child link="Body_RWY"/>
     <axis xyz="0 0 1"/>
-    <limit effort="10.0" lower="-3.14158" upper="3.14158" velocity="1.0"/>
+    <limit effort="50.0" lower="-3.14158" upper="3.14158" velocity="1.0"/>
   </joint>
   <joint name="RWP" type="revolute">
@@ -1398,5 +1398,5 @@
     <child link="Body_RWP"/>
     <axis xyz="0 1 0"/>
-    <limit effort="10.0" lower="-1.64061" upper="1.01229" velocity="1.0"/>
+    <limit effort="50.0" lower="-1.64061" upper="1.01229" velocity="1.0"/>
   </joint>
   <!-- Joints related to fingers on the right hand -->
