Commit message: add the kinect macro parameter "frame_name" again

File: hubo_description/urdf/sensors/kinect_prosilica_camera.gazebo.xacro (robot description, xacro)
@@ -1,5 +1,5 @@
 <?xml version="1.0"?>
 <root xmlns:xacro="http://ros.org/wiki/xacro">
-<xacro:macro name="kinect_ir_gazebo_v0" params="link_name camera_name">
+<xacro:macro name="kinect_ir_gazebo_v0" params="link_name frame_name camera_name">
   <gazebo reference="${link_name}">
     <sensor type="depth" name="${name}_ir_sensor">
@@ -28,5 +28,5 @@
         <depthImageCameraInfoTopicName>/${camera_name}/depth/camera_info</depthImageCameraInfoTopicName>
         <pointCloudTopicName>/${camera_name}/depth/points</pointCloudTopicName>
-        <frameName>${link_name}</frameName>
+        <frameName>${frame_name}</frameName>
         <pointCloudCutoff>0.5</pointCloudCutoff>
         <!-- original values:

File: hubo_description/urdf/sensors/kinect_prosilica_camera.urdf.xacro (robot description, xacro)
@@ -70,5 +70,5 @@
     <!-- gazebo extensions -->
     <!--<xacro:kinect_ir_gazebo_v0 link_name="${name}_kinect_ir_optical_frame" frame_name="projection_frame" camera_name="head_mount_kinect" />-->
-    <xacro:kinect_ir_gazebo_v0 link_name="${name}_kinect_ir_link" camera_name="head_mount_kinect" />
+    <xacro:kinect_ir_gazebo_v0 link_name="${name}_kinect_ir_link" frame_name="${name}_kinect_ir_optical_frame" camera_name="head_mount_kinect" />
     <transmission name="${name}_trans">
       <type>transmission_interface/SimpleTransmission</type>

Commit message: add and use "prosilica camera"

File: hubo_description/urdf/sensors/kinect_prosilica_camera.gazebo.xacro (robot description, xacro)
@@ -97,3 +97,85 @@
 </xacro:macro>
 -->
+<xacro:macro name="prosilica_cam_gazebo_v1" params="link_name frame_name camera_name ">
+  <gazebo reference="${link_name}">
+    <sensor type="camera" name="${link_name}_sensor">
+      <always_on>true</always_on>
+      <update_rate>1.0</update_rate>
+      <camera>
+        <horizontal_fov>${64.2*M_PI/180.0}</horizontal_fov>
+        <image>
+          <format>R8G8B8</format>
+          <width>320</width>
+          <height>240</height>
+        </image>
+        <clip>
+          <near>0.1</near>
+          <far>100</far>
+        </clip>
+      </camera>
+      <plugin name="${link_name}_controller" filename="libgazebo_ros_prosilica.so">
+        <alwaysOn>true</alwaysOn>
+        <updateRate>1.0</updateRate>
+        <cameraName>${camera_name}_1mb</cameraName>
+        <imageTopicName>image_raw</imageTopicName>
+        <cameraInfoTopicName>camera_info</cameraInfoTopicName>
+        <depthImageTopicName>depth/image_raw</depthImageTopicName>
+        <depthImageCameraInfoTopicName>depth/camera_info</depthImageCameraInfoTopicName>
+        <pollServiceName>request_image</pollServiceName>
+        <pointCloudTopicName>points</pointCloudTopicName>
+        <frameName>${frame_name}</frameName>
+        <pointCloudCutoff>0.4</pointCloudCutoff>
+        <distortionK1>0.0</distortionK1>
+        <distortionK2>0.0</distortionK2>
+        <distortionK3>0.0</distortionK3>
+        <distortionT1>0.0</distortionT1>
+        <distortionT2>0.0</distortionT2>
+        <CxPrime>0</CxPrime>
+        <Cx>0</Cx>
+        <Cy>0</Cy>
+        <focalLength>0</focalLength>
+        <hackBaseline>0</hackBaseline>
+      </plugin>
+    </sensor>
+    <sensor type="depth" name="${link_name}_sim_pcd_sensor">
+      <always_on>true</always_on>
+      <update_rate>1.0</update_rate>
+      <camera>
+        <horizontal_fov>${64.2*M_PI/180.0}</horizontal_fov>
+        <image>
+          <format>R8G8B8</format>
+          <width>320</width>
+          <height>240</height>
+        </image>
+        <clip>
+          <near>0.1</near>
+          <far>100</far>
+        </clip>
+      </camera>
+      <plugin name="${link_name}_sim_pcd_controller" filename="libgazebo_ros_openni_kinect.so">
+        <alwaysOn>true</alwaysOn>
+        <updateRate>1.0</updateRate>
+        <cameraName>${camera_name}_1mb_sim_pcd</cameraName>
+        <imageTopicName>image_raw</imageTopicName>
+        <depthImageTopicName>depth/image_raw</depthImageTopicName>
+        <depthImageCameraInfoTopicName>depth/camera_info</depthImageCameraInfoTopicName>
+        <cameraInfoTopicName>camera_info</cameraInfoTopicName>
+        <pointCloudTopicName>points</pointCloudTopicName>
+        <frameName>${frame_name}</frameName>
+        <pointCloudCutoff>0.4</pointCloudCutoff>
+        <distortionK1>0</distortionK1>
+        <distortionK2>0</distortionK2>
+        <distortionK3>0</distortionK3>
+        <distortionT1>0</distortionT1>
+        <distortionT2>0</distortionT2>
+        <CxPrime>0</CxPrime>
+        <Cx>0</Cx>
+        <Cy>0</Cy>
+        <focalLength>0</focalLength>
+        <hackBaseline>0</hackBaseline>
+      </plugin>
+    </sensor>
+    <material value="Gazebo/Red" />
+  </gazebo>
+</xacro:macro>
 </root>

File: hubo_description/urdf/sensors/kinect_prosilica_camera.urdf.xacro (robot description, xacro)
@@ -117,4 +117,41 @@
     <xacro:kinect_rgb_gazebo_v0 link_name="${name}_kinect_rgb_optical_frame" frame_name="${name}_kinect_rgb_optical_frame" camera_name="head_mount_kinect" />
 -->
+    <!-- prosilica sensor physical attachment -->
+    <joint name="${name}_prosilica_joint" type="fixed">
+      <origin xyz="-0.046457 0.0125 0.088921" rpy="0 0 0"/>
+      <parent link="${name}_link"/>
+      <child link="${name}_prosilica_link"/>
+    </joint>
+    <link name="${name}_prosilica_link">
+      <inertial>
+        <mass value="0.1" />
+        <origin xyz="0 0 0" rpy="0 0 0"/>
+        <inertia ixx="0.01"  ixy="0.0"  ixz="0.0"
+                 iyy="0.01"  iyz="0.0"
+                 izz="0.01" />
+      </inertial>
+      <visual>
+        <origin xyz="0.0 0.0 0" rpy="0 0 0"/>
+        <geometry>
+          <sphere radius="0.0005"/>
+        </geometry>
+      </visual>
+      <collision>
+        <origin xyz="0.0 0.0 0" rpy="0 0 0"/>
+        <geometry>
+          <sphere radius="0.0005"/>
+        </geometry>
+      </collision>
+    </link>
+    <!-- prosilica sensor frame -->
+    <joint name="${name}_prosilica_optical_frame_joint" type="fixed">
+      <origin xyz="${cal_high_def_x}            ${cal_high_def_y}         ${cal_high_def_z}"
+                rpy="${-M_PI/2+cal_high_def_roll} ${0.0+cal_high_def_pitch} ${-M_PI/2+cal_high_def_yaw}" />
+      <parent link="${name}_prosilica_link"/>
+      <child link="${name}_prosilica_optical_frame"/>
+    </joint>
+    <link name="${name}_prosilica_optical_frame"/>
+    <!-- gazebo extensions -->
+    <xacro:prosilica_cam_gazebo_v1 link_name="${name}_prosilica_link" camera_name="prosilica_camera" frame_name="${name}_prosilica_optical_frame" />
   </xacro:macro>
 </root>

Commit message: add and use "prosilica camera"

File: hubo_description/urdf/sensors/kinect_prosilica_camera.gazebo.xacro (robot description, xacro)
@@ -97,3 +97,85 @@
 </xacro:macro>
 -->
+<xacro:macro name="prosilica_cam_gazebo_v1" params="link_name frame_name camera_name ">
+  <gazebo reference="${link_name}">
+    <sensor type="camera" name="${link_name}_sensor">
+      <always_on>true</always_on>
+      <update_rate>1.0</update_rate>
+      <camera>
+        <horizontal_fov>${64.2*M_PI/180.0}</horizontal_fov>
+        <image>
+          <format>R8G8B8</format>
+          <width>320</width>
+          <height>240</height>
+        </image>
+        <clip>
+          <near>0.1</near>
+          <far>100</far>
+        </clip>
+      </camera>
+      <plugin name="${link_name}_controller" filename="libgazebo_ros_prosilica.so">
+        <alwaysOn>true</alwaysOn>
+        <updateRate>1.0</updateRate>
+        <cameraName>${camera_name}_1mb</cameraName>
+        <imageTopicName>image_raw</imageTopicName>
+        <cameraInfoTopicName>camera_info</cameraInfoTopicName>
+        <depthImageTopicName>depth/image_raw</depthImageTopicName>
+        <depthImageCameraInfoTopicName>depth/camera_info</depthImageCameraInfoTopicName>
+        <pollServiceName>request_image</pollServiceName>
+        <pointCloudTopicName>points</pointCloudTopicName>
+        <frameName>${frame_name}</frameName>
+        <pointCloudCutoff>0.4</pointCloudCutoff>
+        <distortionK1>0.0</distortionK1>
+        <distortionK2>0.0</distortionK2>
+        <distortionK3>0.0</distortionK3>
+        <distortionT1>0.0</distortionT1>
+        <distortionT2>0.0</distortionT2>
+        <CxPrime>0</CxPrime>
+        <Cx>0</Cx>
+        <Cy>0</Cy>
+        <focalLength>0</focalLength>
+        <hackBaseline>0</hackBaseline>
+      </plugin>
+    </sensor>
+    <sensor type="depth" name="${link_name}_sim_pcd_sensor">
+      <always_on>true</always_on>
+      <update_rate>1.0</update_rate>
+      <camera>
+        <horizontal_fov>${64.2*M_PI/180.0}</horizontal_fov>
+        <image>
+          <format>R8G8B8</format>
+          <width>320</width>
+          <height>240</height>
+        </image>
+        <clip>
+          <near>0.1</near>
+          <far>100</far>
+        </clip>
+      </camera>
+      <plugin name="${link_name}_sim_pcd_controller" filename="libgazebo_ros_openni_kinect.so">
+        <alwaysOn>true</alwaysOn>
+        <updateRate>1.0</updateRate>
+        <cameraName>${camera_name}_1mb_sim_pcd</cameraName>
+        <imageTopicName>image_raw</imageTopicName>
+        <depthImageTopicName>depth/image_raw</depthImageTopicName>
+        <depthImageCameraInfoTopicName>depth/camera_info</depthImageCameraInfoTopicName>
+        <cameraInfoTopicName>camera_info</cameraInfoTopicName>
+        <pointCloudTopicName>points</pointCloudTopicName>
+        <frameName>${frame_name}</frameName>
+        <pointCloudCutoff>0.4</pointCloudCutoff>
+        <distortionK1>0</distortionK1>
+        <distortionK2>0</distortionK2>
+        <distortionK3>0</distortionK3>
+        <distortionT1>0</distortionT1>
+        <distortionT2>0</distortionT2>
+        <CxPrime>0</CxPrime>
+        <Cx>0</Cx>
+        <Cy>0</Cy>
+        <focalLength>0</focalLength>
+        <hackBaseline>0</hackBaseline>
+      </plugin>
+    </sensor>
+    <material value="Gazebo/Red" />
+  </gazebo>
+</xacro:macro>
 </root>

File: hubo_description/urdf/sensors/kinect_prosilica_camera.urdf.xacro (robot description, xacro)
@@ -100,4 +100,41 @@
     <xacro:kinect_rgb_gazebo_v0 link_name="${name}_kinect_rgb_optical_frame" frame_name="${name}_kinect_rgb_optical_frame" camera_name="head_mount_kinect" />
 -->
+    <!-- prosilica sensor physical attachment -->
+    <joint name="${name}_prosilica_joint" type="fixed">
+      <origin xyz="-0.046457 0.0125 0.088921" rpy="0 0 0"/>
+      <parent link="${name}_link"/>
+      <child link="${name}_prosilica_link"/>
+    </joint>
+    <link name="${name}_prosilica_link">
+      <inertial>
+        <mass value="0.1" />
+        <origin xyz="0 0 0" rpy="0 0 0"/>
+        <inertia ixx="0.01"  ixy="0.0"  ixz="0.0"
+                 iyy="0.01"  iyz="0.0"
+                 izz="0.01" />
+      </inertial>
+      <visual>
+        <origin xyz="0.0 0.0 0" rpy="0 0 0"/>
+        <geometry>
+          <sphere radius="0.0005"/>
+        </geometry>
+      </visual>
+      <collision>
+        <origin xyz="0.0 0.0 0" rpy="0 0 0"/>
+        <geometry>
+          <sphere radius="0.0005"/>
+        </geometry>
+      </collision>
+    </link>
+    <!-- prosilica sensor frame -->
+    <joint name="${name}_prosilica_optical_frame_joint" type="fixed">
+      <origin xyz="${cal_high_def_x}            ${cal_high_def_y}         ${cal_high_def_z}"
+                rpy="${-M_PI/2+cal_high_def_roll} ${0.0+cal_high_def_pitch} ${-M_PI/2+cal_high_def_yaw}" />
+      <parent link="${name}_prosilica_link"/>
+      <child link="${name}_prosilica_optical_frame"/>
+    </joint>
+    <link name="${name}_prosilica_optical_frame"/>
+    <!-- gazebo extensions -->
+    <xacro:prosilica_cam_gazebo_v1 link_name="${name}_prosilica_link" camera_name="prosilica_camera" frame_name="${name}_prosilica_optical_frame" />
   </xacro:macro>
 </root>
