Commit message: add debugging joint controller & transmission

File: hubo_description/urdf/sensors/kinect_prosilica_camera.urdf.xacro (robot description, xacro)
@@ -8,9 +8,11 @@
   <xacro:macro name="kinect_prosilica_camera_swept_back_v0" params="name parent *origin">
     <!-- stl contains structure + kinect + prosilica combo -->
-    <joint name="${name}_joint" type="fixed">
+    <joint name="${name}_joint" type="revolute">
       <!-- <limit lower="0.1" upper="0.1" effort="10000" velocity="100.0"/> -->
       <insert_block name="origin" />
       <parent link="${parent}"/>
       <child link="${name}_link"/>
+      <axis xyz="0 1 0"/>
+      <limit effort="10.0" lower="-3.14158" upper="3.14158" velocity="1.0"/>
     </joint>
     <link name="${name}_link">
@@ -60,6 +62,21 @@
     </joint>
     <link name="${name}_kinect_ir_optical_frame"/>
+    <joint name="projection_joint" type="fixed">
+      <origin xyz="0 0 0" rpy="${M_PI/2.0} ${-M_PI/2.0} 0" />
+      <parent link="${name}_kinect_ir_optical_frame"/>
+      <child link="projection_frame"/>
+    </joint>
+    <link name="projection_frame"/>
     <!-- gazebo extensions -->
+    <!--<xacro:kinect_ir_gazebo_v0 link_name="${name}_kinect_ir_optical_frame" frame_name="projection_frame" camera_name="head_mount_kinect" />-->
     <xacro:kinect_ir_gazebo_v0 link_name="${name}_kinect_ir_optical_frame" camera_name="head_mount_kinect" />
+    <transmission name="${name}_trans">
+      <type>transmission_interface/SimpleTransmission</type>
+      <joint name="${name}_joint" />
+      <actuator name="${name}_motor">
+          <hardwareInterface>EffortJointInterface</hardwareInterface>
+          <mechanicalReduction>1</mechanicalReduction>
+      </actuator>
+    </transmission>
 <!--
     // kinect rgb sensor physical attachment

Commit message: attach the prosilica using two perpendicular joints

File: hubo_description/urdf/sensors/kinect_prosilica_camera.urdf.xacro (robot description, xacro)
@@ -128,11 +128,52 @@
     </link>
     <!-- prosilica sensor frame -->
-    <joint name="${name}_prosilica_optical_frame_joint" type="fixed">
-      <origin xyz="${cal_high_def_x}            ${cal_high_def_y}         ${cal_high_def_z}"
-                rpy="${-M_PI/2+cal_high_def_roll} ${0.0+cal_high_def_pitch} ${-M_PI/2+cal_high_def_yaw}" />
+    <joint name="${name}_prosilica_optical_frame_joint1" type="revolute">
+      <origin xyz="0 0 0" rpy="0 0 0" />
+      <axis xyz="0 1 0" />
+      <limit effort="10.0" lower="-3.14158" upper="3.14158" velocity="1.0"/>
       <parent link="${name}_prosilica_link"/>
+      <child link="${name}_prosilica_frame1"/>
+    </joint>
+    <link name="${name}_prosilica_frame1">
+      <inertial>
+        <mass value="0.01" />
+        <origin xyz="0 0 0" rpy="0 0 0"/>
+        <inertia ixx="0.001"  ixy="0.0"  ixz="0.0"
+                 iyy="0.001"  iyz="0.0"
+                 izz="0.001" />
+      </inertial>
+    </link>
+    <joint name="${name}_prosilica_optical_frame_joint" type="revolute">
+      <origin xyz="0 0 0" rpy="0 0 0" />
+      <axis xyz="1 0 0" />
+      <limit effort="10.0" lower="-3.14158" upper="3.14158" velocity="1.0"/>
+      <parent link="${name}_prosilica_frame1"/>
       <child link="${name}_prosilica_optical_frame"/>
     </joint>
-    <link name="${name}_prosilica_optical_frame"/>
+    <transmission name="${name}_trans1">
+      <type>transmission_interface/SimpleTransmission</type>
+      <joint name="${name}_prosilica_optical_frame_joint1" />
+      <actuator name="${name}_motor1">
+          <hardwareInterface>EffortJointInterface</hardwareInterface>
+          <mechanicalReduction>1</mechanicalReduction>
+      </actuator>
+    </transmission>
+    <transmission name="${name}_trans2">
+      <type>transmission_interface/SimpleTransmission</type>
+      <joint name="${name}_prosilica_optical_frame_joint" />
+      <actuator name="${name}_motor2">
+          <hardwareInterface>EffortJointInterface</hardwareInterface>
+          <mechanicalReduction>1</mechanicalReduction>
+      </actuator>
+    </transmission>
+    <link name="${name}_prosilica_optical_frame">
+      <inertial>
+        <mass value="0.01" />
+        <origin xyz="0 0 0" rpy="0 0 0"/>
+        <inertia ixx="0.001"  ixy="0.0"  ixz="0.0"
+                 iyy="0.001"  iyz="0.0"
+                 izz="0.001" />
+      </inertial>
+    </link>
     <!-- gazebo extensions -->
     <xacro:prosilica_cam_gazebo_v1 link_name="${name}_prosilica_link" camera_name="prosilica_camera" frame_name="${name}_prosilica_optical_frame" />

Commit message: add another 2 joints to facilitate finding the proper sensor position

File: hubo_description/urdf/sensors/kinect_prosilica_camera.urdf.xacro (robot description, xacro)
@@ -101,6 +101,9 @@
 -->
     <!-- prosilica sensor physical attachment -->
-    <joint name="${name}_prosilica_joint" type="fixed">
+    <joint name="${name}_prosilica_joint" type="revolute">
+      <!-- thought this would make it work the way i want to <origin xyz="-0.046457 0.0125 0.088921" rpy="0 ${-M_PI/2.0} 0"/>-->
       <origin xyz="-0.046457 0.0125 0.088921" rpy="0 0 0"/>
+      <axis xyz="0 1 0" />
+      <limit effort="10.0" lower="-3.14158" upper="3.14158" velocity="1.0"/>
       <parent link="${name}_link"/>
       <child link="${name}_prosilica_link"/>
@@ -128,9 +131,25 @@
     </link>
     <!-- prosilica sensor frame -->
+    <joint name="${name}_prosilica_optical_frame_joint_z" type="revolute">
+      <origin xyz="0 0 0" rpy="0 0 0" />
+      <axis xyz="0 0 1" />
+      <limit effort="10.0" lower="-3.14158" upper="3.14158" velocity="1.0"/>
+      <parent link="${name}_prosilica_link"/>
+      <child link="${name}_prosilica_link_z"/>
+    </joint>
+    <link name="${name}_prosilica_link_z">
+      <inertial>
+        <mass value="0.01" />
+        <origin xyz="0 0 0" rpy="0 0 0"/>
+        <inertia ixx="0.001"  ixy="0.0"  ixz="0.0"
+                 iyy="0.001"  iyz="0.0"
+                 izz="0.001" />
+      </inertial>
+    </link>
     <joint name="${name}_prosilica_optical_frame_joint1" type="revolute">
       <origin xyz="0 0 0" rpy="0 0 0" />
       <axis xyz="0 1 0" />
       <limit effort="10.0" lower="-3.14158" upper="3.14158" velocity="1.0"/>
-      <parent link="${name}_prosilica_link"/>
+      <parent link="${name}_prosilica_link_z"/>
       <child link="${name}_prosilica_frame1"/>
     </joint>
@@ -151,4 +170,20 @@
       <child link="${name}_prosilica_optical_frame"/>
     </joint>
+    <transmission name="${name}_trans0">
+      <type>transmission_interface/SimpleTransmission</type>
+      <joint name="${name}_prosilica_joint" />
+      <actuator name="${name}_motor0">
+          <hardwareInterface>EffortJointInterface</hardwareInterface>
+          <mechanicalReduction>1</mechanicalReduction>
+      </actuator>
+    </transmission>
+    <transmission name="${name}_trans_z">
+      <type>transmission_interface/SimpleTransmission</type>
+      <joint name="${name}_prosilica_optical_frame_joint_z" />
+      <actuator name="${name}_motor_z">
+          <hardwareInterface>EffortJointInterface</hardwareInterface>
+          <mechanicalReduction>1</mechanicalReduction>
+      </actuator>
+    </transmission>
     <transmission name="${name}_trans1">
       <type>transmission_interface/SimpleTransmission</type>

Commit message: fix prosilica sensor location

File: hubo_description/urdf/sensors/kinect_prosilica_camera.urdf.xacro (robot description, xacro)
@@ -103,5 +103,5 @@
     <joint name="${name}_prosilica_joint" type="revolute">
       <!-- thought this would make it work the way i want to <origin xyz="-0.046457 0.0125 0.088921" rpy="0 ${-M_PI/2.0} 0"/>-->
-      <origin xyz="-0.046457 0.0125 0.088921" rpy="0 0 0"/>
+      <origin xyz="0 0 0" rpy="0 0 0"/>
       <axis xyz="0 1 0" />
       <limit effort="10.0" lower="-3.14158" upper="3.14158" velocity="1.0"/>
