Commit message: kinect now works but looks downwards

File: hubo_description/robots/hubo_with_kinect.urdf.xacro (robot description, xacro)
@@ -16,8 +16,6 @@
   <!-- Kinect -->
   <xacro:kinect_prosilica_camera_swept_back_v0 name="hand_mount" parent="Body_RWP" >
-    <!-- <origin xyz="0 0 0" rpy="0 1.570796 0"/> -->
-    <!-- <origin xyz="0.032267 -0.0125 -0.136453" rpy="0 0 0"/> -->
-    <!-- <origin xyz="0.032267 -0.0125 -0.25" rpy="0 1.570796 0"/> -->
-    <origin xyz="0 0 -0.15" rpy="0 1.570796 0"/>
+    <!--<origin xyz="0 0.005 -0.15" rpy="1.570796 1.570796 0"/>-->
+    <origin xyz="0 -2 -0.15" rpy="1.570796 1.570796 0"/>
   </xacro:kinect_prosilica_camera_swept_back_v0>
 </robot>

File: hubo_description/urdf/hubo.urdf.xacro (robot description, xacro)
@@ -5,4 +5,10 @@
        xmlns:xacro="http://ros.org/wiki/xacro">
 <xacro:macro name="hubo">
+  <!-- Used to fix the hubo to the Gazebo World -->
+  <link name="world"/>
+  <joint name="fixTheHuboToWorld" type="fixed">
+    <parent link="world"/>
+    <child link="Body_Torso"/>
+  </joint>
   <link name="Body_Torso">
     <inertial>
@@ -1797,9 +1803,4 @@
     </plugin>
   </gazebo>
-  <!-- model pose -->
-  <gazebo>
-    <!-- robot model offset -->
-    <pose>0 0 1 0 0 0</pose>
-  </gazebo>
 </xacro:macro>
 </robot>

File: hubo_description/urdf/sensors/kinect_prosilica_camera.gazebo.xacro (robot description, xacro)
@@ -1,5 +1,5 @@
 <?xml version="1.0"?>
 <root xmlns:xacro="http://ros.org/wiki/xacro">
-<xacro:macro name="kinect_ir_gazebo_v0" params="link_name frame_name camera_name">
+<xacro:macro name="kinect_ir_gazebo_v0" params="link_name camera_name">
   <gazebo reference="${link_name}">
     <sensor type="depth" name="${name}_ir_sensor">
@@ -28,5 +28,5 @@
         <depthImageCameraInfoTopicName>/${camera_name}/depth/camera_info</depthImageCameraInfoTopicName>
         <pointCloudTopicName>/${camera_name}/depth/points</pointCloudTopicName>
-        <frameName>${frame_name}</frameName>
+        <frameName>${link_name}</frameName>
         <pointCloudCutoff>0.5</pointCloudCutoff>
         <!-- original values:
@@ -52,4 +52,5 @@
   </gazebo>
 </xacro:macro>
+<!--
 <xacro:macro name="kinect_rgb_gazebo_v0" params="link_name frame_name camera_name">
   <gazebo reference="${link_name}">
@@ -78,11 +79,11 @@
         <depthImageCameraInfoTopicName>/${camera_name}/depth/camera_info</depthImageCameraInfoTopicName>
         <pointCloudTopicName>/${camera_name}/depth_registered/points</pointCloudTopicName>
-        <frameName>${frame_name}</frameName>
+        <frameName>${link_name}</frameName>
         <pointCloudCutoff>0.5</pointCloudCutoff>
-        <distortionK1>0.00000001</distortionK1>
-        <distortionK2>0.00000001</distortionK2>
-        <distortionK3>0.00000001</distortionK3>
-        <distortionT1>0.00000001</distortionT1>
-        <distortionT2>0.00000001</distortionT2>
+        <distortionK1>0</distortionK1>
+        <distortionK2>0</distortionK2>
+        <distortionK3>0</distortionK3>
+        <distortionT1>0</distortionT1>
+        <distortionT2>0</distortionT2>
         <CxPrime>0</CxPrime>
         <Cx>0</Cx>
@@ -95,100 +96,4 @@
   </gazebo>
 </xacro:macro>
-<xacro:macro name="kinect_prosilica_gazebo" params="joint_name link_name">
-  <gazebo>
-    <plugin name="${link_name}_srp_controller" filename="libgazebo_ros_srp.so">
-      <bodyName>${link_name}</bodyName>
-      <jointName>${joint_name}</jointName>
-      <topicName>${link_name}</topicName>
-    </plugin>
-  </gazebo>
-  <!-- also add transmission for this sliding joint -->
-  <transmission type="pr2_mechanism_model/SimpleTransmission" name="${joint_name}_trans">
-    <actuator name="${joint_name}_motor" />
-    <joint name="${joint_name}" />
-    <mechanicalReduction>1</mechanicalReduction>
-  </transmission>
-</xacro:macro>
-<xacro:macro name="prosilica_cam_gazebo_v1" params="link_name frame_name camera_name ">
-  <gazebo reference="${link_name}">
-    <sensor type="camera" name="${link_name}_sensor">
-      <always_on>true</always_on>
-      <update_rate>1.0</update_rate>
-      <camera>
-        <horizontal_fov>${64.2*M_PI/180.0}</horizontal_fov>
-        <image>
-          <format>R8G8B8</format>
-          <width>320</width>
-          <height>240</height>
-        </image>
-        <clip>
-          <near>0.1</near>
-          <far>100</far>
-        </clip>
-      </camera>
-      <plugin name="${link_name}_controller" filename="libgazebo_ros_prosilica.so">
-        <alwaysOn>true</alwaysOn>
-        <updateRate>1.0</updateRate>
-        <cameraName>${camera_name}_1mb</cameraName>
-        <imageTopicName>image_raw</imageTopicName>
-        <cameraInfoTopicName>camera_info</cameraInfoTopicName>
-        <depthImageTopicName>depth/image_raw</depthImageTopicName>
-        <depthImageCameraInfoTopicName>depth/camera_info</depthImageCameraInfoTopicName>
-        <pollServiceName>request_image</pollServiceName>
-        <pointCloudTopicName>points</pointCloudTopicName>
-        <frameName>${frame_name}</frameName>
-        <pointCloudCutoff>0.4</pointCloudCutoff>
-        <distortionK1>0.0</distortionK1>
-        <distortionK2>0.0</distortionK2>
-        <distortionK3>0.0</distortionK3>
-        <distortionT1>0.0</distortionT1>
-        <distortionT2>0.0</distortionT2>
-        <CxPrime>0</CxPrime>
-        <Cx>0</Cx>
-        <Cy>0</Cy>
-        <focalLength>0</focalLength>
-        <hackBaseline>0</hackBaseline>
-      </plugin>
-    </sensor>
-    <sensor type="depth" name="${link_name}_sim_pcd_sensor">
-      <always_on>true</always_on>
-      <update_rate>1.0</update_rate>
-      <camera>
-        <horizontal_fov>${64.2*M_PI/180.0}</horizontal_fov>
-        <image>
-          <format>R8G8B8</format>
-          <width>320</width>
-          <height>240</height>
-        </image>
-        <clip>
-          <near>0.1</near>
-          <far>100</far>
-        </clip>
-      </camera>
-      <plugin name="${link_name}_sim_pcd_controller" filename="libgazebo_ros_openni_kinect.so">
-        <alwaysOn>true</alwaysOn>
-        <updateRate>1.0</updateRate>
-        <cameraName>${camera_name}_1mb_sim_pcd</cameraName>
-        <imageTopicName>image_raw</imageTopicName>
-        <depthImageTopicName>depth/image_raw</depthImageTopicName>
-        <depthImageCameraInfoTopicName>depth/camera_info</depthImageCameraInfoTopicName>
-        <cameraInfoTopicName>camera_info</cameraInfoTopicName>
-        <pointCloudTopicName>points</pointCloudTopicName>
-        <frameName>${frame_name}</frameName>
-        <pointCloudCutoff>0.4</pointCloudCutoff>
-        <distortionK1>0.00000001</distortionK1>
-        <distortionK2>0.00000001</distortionK2>
-        <distortionK3>0.00000001</distortionK3>
-        <distortionT1>0.00000001</distortionT1>
-        <distortionT2>0.00000001</distortionT2>
-        <CxPrime>0</CxPrime>
-        <Cx>0</Cx>
-        <Cy>0</Cy>
-        <focalLength>0</focalLength>
-        <hackBaseline>0</hackBaseline>
-      </plugin>
-    </sensor>
-    <material value="Gazebo/Red" />
-  </gazebo>
-</xacro:macro>
+-->
 </root>

File: hubo_description/urdf/sensors/kinect_prosilica_camera.urdf.xacro (robot description, xacro)
@@ -5,5 +5,4 @@
       xmlns:xacro="http://ros.org/wiki/xacro">
   <xacro:include filename="$(find hubo_description)/urdf/sensors/kinect_prosilica_camera.gazebo.xacro" />
-  <property name="ir_depth_rgb_offset_y" value="0.01"/> <!-- FIXME: what is this offset? -->
   <!-- kinect and prosilica combo -->
   <xacro:macro name="kinect_prosilica_camera_swept_back_v0" params="name parent *origin">
@@ -12,5 +11,4 @@
       <!-- <limit lower="0.1" upper="0.1" effort="10000" velocity="100.0"/> -->
       <insert_block name="origin" />
-      <!-- <origin xyz="-0.138 0 0.091" rpy="0 0 0"/> -->
       <parent link="${parent}"/>
       <child link="${name}_link"/>
@@ -33,19 +31,8 @@
         </material>
       </visual>
-      <collision>
-        <origin xyz="0.0 0.0 0" rpy="0 0 0"/>
-        <geometry>
-          <sphere radius="0.0005"/>
-        </geometry>
-      </collision>
     </link>
-    <!-- plugin for updating structure pose \
-    <xacro:kinect_prosilica_gazebo joint_name="${name}_kinect_prosilica_joint"
-                                   link_name="${name}_kinect_prosilica_link" />
-    -->
     <!-- kinect ir sensor physical attachment -->
     <joint name="${name}_kinect_ir_joint" type="fixed">
-      <!-- <origin xyz="-0.032267 0.0125 0.136453" rpy="0 0 0"/> -->
-      <origin xyz="0 0 0" rpy="0 0 0"/>
+      <origin xyz="0 0 0" rpy="0 ${M_PI/2.0} 0"/>
       <parent link="${name}_link"/>
       <child link="${name}_kinect_ir_link"/>
@@ -62,18 +49,11 @@
         <origin xyz="0.0 0.0 0" rpy="0 0 0"/>
         <geometry>
-          <sphere radius="0.0005"/>
+          <sphere radius="0.005"/>
         </geometry>
       </visual>
-      <collision>
-        <origin xyz="0.0 0.0 0" rpy="0 0 0"/>
-        <geometry>
-          <sphere radius="0.0005"/>
-        </geometry>
-      </collision>
     </link>
     <!-- kinect ir sensor frame -->
     <joint name="${name}_kinect_ir_optical_frame_joint" type="fixed">
-      <origin xyz="${cal_kinect_x}            ${cal_kinect_y + ir_depth_rgb_offset_y}         ${cal_kinect_z}"
-                rpy="${-M_PI/2+cal_kinect_roll} ${0.0+cal_kinect_pitch} ${-M_PI/2+cal_kinect_yaw}" />
+      <origin xyz="0 0 0" rpy="0 ${M_PI/2.0} 0" />
       <parent link="${name}_kinect_ir_link"/>
       <child link="${name}_kinect_ir_optical_frame"/>
@@ -81,6 +61,7 @@
     <link name="${name}_kinect_ir_optical_frame"/>
     <!-- gazebo extensions -->
-    <xacro:kinect_ir_gazebo_v0 link_name="${name}_kinect_ir_link" frame_name="${name}_kinect_ir_optical_frame" camera_name="head_mount_kinect" />
-    <!-- kinect rgb sensor physical attachment -->
+    <xacro:kinect_ir_gazebo_v0 link_name="${name}_kinect_ir_optical_frame" camera_name="head_mount_kinect" />
+<!--
+    // kinect rgb sensor physical attachment
     <joint name="${name}_kinect_rgb_joint" type="fixed">
       <origin xyz="0 -0.03 0" rpy="0 0 0"/>
@@ -99,5 +80,5 @@
         <origin xyz="0.0 0.0 0" rpy="0 0 0"/>
         <geometry>
-          <sphere radius="0.0005"/>
+          <sphere radius="0.005"/>
         </geometry>
       </visual>
@@ -109,14 +90,14 @@
       </collision>
     </link>
-    <!-- kinect rgb sensor frame -->
+    // kinect rgb sensor frame
     <joint name="${name}_kinect_rgb_optical_frame_joint" type="fixed">
-      <origin xyz="${cal_kinect_x}            ${cal_kinect_y}         ${cal_kinect_z}"
-                rpy="${-M_PI/2+cal_kinect_roll} ${0.0+cal_kinect_pitch} ${-M_PI/2+cal_kinect_yaw}" />
+      <origin xyz="0 0 0" rpy="0 ${-M_PI/2.0} 0" />
       <parent link="${name}_kinect_rgb_link"/>
       <child link="${name}_kinect_rgb_optical_frame"/>
     </joint>
     <link name="${name}_kinect_rgb_optical_frame"/>
-    <!-- gazebo extensions -->
-    <xacro:kinect_rgb_gazebo_v0 link_name="${name}_kinect_rgb_link" frame_name="${name}_kinect_rgb_optical_frame" camera_name="head_mount_kinect" />
+    // gazebo extensions
+    <xacro:kinect_rgb_gazebo_v0 link_name="${name}_kinect_rgb_optical_frame" frame_name="${name}_kinect_rgb_optical_frame" camera_name="head_mount_kinect" />
+-->
   </xacro:macro>
 </root>

Commit message: add a comment documenting what the original position of kinect was

File: hubo_description/robots/hubo_with_kinect.urdf.xacro (robot description, xacro)
@@ -16,6 +16,6 @@
   <!-- Kinect -->
   <xacro:kinect_prosilica_camera_swept_back_v0 name="hand_mount" parent="Body_RWP" >
-    <!--<origin xyz="0 0.005 -0.15" rpy="1.570796 1.570796 0"/>-->
-    <origin xyz="0 -2 -0.15" rpy="1.570796 1.570796 0"/>
+    <!-- This is the original position of the kinect: <origin xyz="0 0.005 -0.15" rpy="1.570796 1.570796 0"/>-->
+    <origin xyz="0 -2 -0.15" rpy="${M_PI/2.0} ${M_PI/2.0} 0"/>
   </xacro:kinect_prosilica_camera_swept_back_v0>
 </robot>

Commit message: return the sensor to Hubo's right hand

File: hubo_description/robots/hubo_with_kinect.urdf.xacro (robot description, xacro)
@@ -16,6 +16,5 @@
   <!-- Kinect -->
   <xacro:kinect_prosilica_camera_swept_back_v0 name="hand_mount" parent="Body_RWP" >
-    <!-- This is the original position of the kinect: <origin xyz="0 0.005 -0.15" rpy="1.570796 1.570796 0"/>-->
-    <origin xyz="0 -2 -0.15" rpy="${M_PI/2.0} ${M_PI/2.0} 0"/>
+    <origin xyz="0 0.005 -0.15" rpy="${M_PI/2.0} ${M_PI/2.0} 0"/>
   </xacro:kinect_prosilica_camera_swept_back_v0>
 </robot>

Commit message: return the sensor to Hubo's right hand where it belongs

File: hubo_description/robots/hubo_with_kinect.urdf.xacro (robot description, xacro)
@@ -16,6 +16,5 @@
   <!-- Kinect -->
   <xacro:kinect_prosilica_camera_swept_back_v0 name="hand_mount" parent="Body_RWP" >
-    <!--<origin xyz="0 0.005 -0.15" rpy="1.570796 1.570796 0"/>-->
-    <origin xyz="0 -2 -0.15" rpy="1.570796 1.570796 0"/>
+    <origin xyz="0 0.005 -0.15" rpy="${M_PI/2.0} ${M_PI/2.0} 0"/>
   </xacro:kinect_prosilica_camera_swept_back_v0>
 </robot>
